File: sch_doc/aydongle/aydongle.kicad_pcb (KiCad board)
At the start: 2 copper layers, 53 parts, among them J1 prog, J2 USB_A, J3 Display, J4 Audio-Jack-3, Q1 Q_Photo_NPN_EC, Q2 Q_Photo_NPN_CE, U1 AP1117-33, U2 STM32F103C8TxSmall, U3 YM2149F, U4 LM4811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

Commit message: доделал схему, надеюсь окончательный вариант
Parts:
- removed C25: 0.1uF, Capacitor_SMD:C_0603_1608Metric
- removed R13: 560k, Resistor_SMD:R_0805_2012Metric
- moved C7 2.87 mm to (107.5, 85.1), turned to 0 degrees
- moved C9 1.30 mm to (99.8, 73.1), turned to 180 degrees
- moved C4 1.25 mm to (107.7, 64.8)
- moved C5 0.84 mm to (107.3, 67.3)
- moved R10 0.80 mm to (102.2, 53.5)
- moved C16 0.76 mm to (105.8, 53.5)
- moved C15 0.55 mm to (104.0, 53.4)
- moved Y1 0.53 mm to (103.1, 67.8)
- moved C20 0.52 mm to (104.0, 50.1)
- moved C17 0.50 mm to (107.5, 53.4)
- moved C10 0.45 mm to (105.3, 71.5)
- moved C6 0.45 mm to (103.5, 71.5)
- moved C19 0.40 mm to (100.6, 61.2)
- moved C14 0.39 mm to (111.0, 48.5)
- moved C18 0.37 mm to (98.0, 59.1)
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Connections:
- J3 pad 9: Net-(C25-Pad2) -> /D_RST
- U2 pad 41: (no net) -> /D_RST
Routing:
- net /D_RST: track 0.00 -> 29.2 mm
- net +3V3: track 58.9 -> 47.2 mm
- net GND: track 385.1 -> 395.3 mm
- net Net-(C25-Pad2): track 9.15 -> 0.00 mm
- net Net-(C4-Pad2): track 15.2 -> 16.7 mm
- net /DM: track 25.5 -> 24.2 mm
- net /CLOCK: track 19.8 -> 21.0 mm
- net /RESET: track 16.4 -> 17.5 mm
- net Net-(J3-Pad12): track 7.83 -> 6.84 mm
- net Net-(C5-Pad2): track 13.7 -> 12.8 mm
- net /DA0: track 18.1 -> 18.9 mm
- net /DA2: track 12.8 -> 12.1 mm
- net /DA3: track 10.4 -> 9.74 mm
- net /DA4: track 9.05 -> 8.40 mm
- net /DA1: track 15.9 -> 15.4 mm
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
Commit message: ---
Parts:
- moved C21 89.3 mm to (100.1, 133.1), turned to 90 degrees
- moved C23 88.2 mm to (89.0, 132.2), turned to 0 degrees
- moved U4 87.1 mm to (96.0, 131.8), turned to 180 degrees
- moved J4 86.3 mm to (96.2, 131.5), turned to 270 degrees
- moved C14 83.3 mm to (87.1, 128.3), turned to 270 degrees
- moved C22 83.2 mm to (102.2, 129.9), turned to 90 degrees
- moved R12 82.3 mm to (93.3, 129.2), turned to 180 degrees
- moved C11 80.0 mm to (87.1, 126.5), turned to 90 degrees
- moved C20 77.2 mm to (94.2, 126.7), turned to 270 degrees
- moved C17 72.1 mm to (90.7, 123.4), turned to 90 degrees
- moved U3 71.5 mm to (102.3, 124.0), turned to 180 degrees
- moved C16 71.0 mm to (92.4, 123.3), turned to 90 degrees
- moved C15 70.8 mm to (94.2, 123.4), turned to 90 degrees
- moved R10 70.1 mm to (95.9, 123.3), turned to 270 degrees
- moved C13 67.9 mm to (99.5, 122.9), turned to 180 degrees
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Routing:
- net GND: track 395.3 -> 401.4 mm
- net Net-(C23-Pad1): track 6.56 -> 8.58 mm
- net Net-(C12-Pad1): track 13.3 -> 15.2 mm
- net Net-(C13-Pad1): track 21.0 -> 19.3 mm
- net Net-(C23-Pad2): track 4.33 -> 3.21 mm
- net /SWCLK: track 14.9 -> 15.7 mm
- net /A_CLK: track 49.8 -> 50.5 mm
- net +5V: track 83.0 -> 82.4 mm
- net /PHOT_R: track 9.27 -> 9.79 mm
